File: KiCAD_Proj (ESP32).kicad_pcb (KiCad board)
At the start: 4 copper layers, 31 x 56.9 mm, 35 parts, among them J1 USB_B_Micro, J2 Conn_01x19_Pin, J3 Conn_01x19_Pin, Q1 MMSS8050-H-TP, Q2 MMSS8050-H-TP, SW1 SW_Push, SW2 SW_Push, U1 CP2102N-A01-GQFN28, U2 AMS1117-3.3

Commit message: Finished the schematic diagram and PCB board
Parts:
- added REF**: KiCad-Logo2_5mm_SilkScreen, Symbol:KiCad-Logo2_5mm_SilkScreen, B.Cu at (138.3, 81.0)
- moved G*** 21.3 mm to (138.7, 95.1), turned to -90 degrees
