File: KiCAD_Proj (ESP32).kicad_sch (KiCad schematic)
At the start: 34 parts, among them J1 USB_B_Micro, J2 Conn_01x19_Pin, J3 Conn_01x19_Pin, Q1 MMSS8050-H-TP, Q2 MMSS8050-H-TP, SW1 SW_Push, SW2 SW_Push, U1 CP2102N-A01-GQFN28, U2 AMS1117-3.3, U3 ESP32-WROOM-32

Commit message: Finished the schematic diagram and PCB board
Other:
- company: (none) -> LAUDE, RUSELLE RAE D.
- title: (none) -> ESP32
Changed lines of the file:
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@@
 	(generator_version "9.0")
 	(paper "A4")
+	(title_block
+		(title "ESP32")
+		(company "LAUDE, RUSELLE RAE D.")
+		(comment 1 "ORGANIZATION OF ELECTRONICS ENGINEERING STUDENT")
+		(comment 2 "ELECTRONICS ENGINEERING DEPARTMENT")
+		(comment 3 "COLLEGE OF ENGINEERING")
+		(comment 4 "TECHNOLOGICAL UNIVERSITY OF THE PHILIPPINES")
+	)
 	(text "Switch button"
 		(exclude_from_sim no)
